File: docs/kicad/pcb3.1/pcb.kicad_pcb (KiCad board)
At the start: 2 copper layers, 62.2 x 76.2 mm, 24 parts, among them J1 power, J2 coil1, J3 coil2, J5 Sensor, J8 leds, SW1 SW, SW2 SW, U1 L293D, U2 ESP32_DEV_0

Commit message: build 3 x v3.2
Parts:
- C2: footprint 0_my_footprints:CP_my470uf -> 0_my_footprints:CP_my100uf
- moved C2 1.94 mm to (40.6, -53.1)
